File: pcb/mcguitarpedal/_autosave-mcguitarpedal.kicad_sch (KiCad schematic)
At the start: 74 parts, among them J1 IN, J10 ENCODER2, J11 ENCODER3, J2 PREAMP_HEADERS, J3 BTN_MTX, J4 OUT, J5 EXP, J6 ILI9488 Module, J7 PWR_IN, J8 POT_HP_VOLUME_10k, J9 ENCODER1, Q1 2N3904, Q2 BC416, SW1 SW_BYPASS, SW2 SW_TUNER, SW3 SW_PRESET, SW5 SW_PWR, U1 Teensy4.1, U2 Teensy Audio Board, U4 74HC148, U6 STPDWN-3P-5V, U7 STDN-3A24-ADJ, U8 74HCT595D

Commit message: Rearranged pullups
Parts:
- C9: footprint Capacitor_THT:C_Rect_L7.2mm_W2.5mm_P5.00mm_FKS2_FKP2_MKS2_MKP2 -> Capacitor_SMD:C_1206_3216Metric_Pad1.33x1.80mm_HandSolder
Changed lines of the file:
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@@
 			)
 		)
-		(property "Footprint" "Capacitor_THT:C_Rect_L7.2mm_W2.5mm_P5.00mm_FKS2_FKP2_MKS2_MKP2"
+		(property "Footprint" "Capacitor_SMD:C_1206_3216Metric_Pad1.33x1.80mm_HandSolder"
 			(at 94.9452 12.7 0)
 			(effects
